Commit message: feat: 修改了gazebo仿真中轮椅和kinova的相对位置

File: src/kinova_description/urdf/j2s7s300_with_chair.xacro (robot description, xacro)
@@ -15,9 +15,13 @@
 	xmlns:xacro="http://www.ros.org/wiki/xacro" name="j2s7s300">
   <xacro:property name="M_PI" value="3.1415926"/>
-  <!-- root link, on the ground just below the model origin -->
-  <link name="base_footprint">
-  </link>
+  <link name="base_footprint"/>
+  <joint name="connect_root_and_wheelchair" type="fixed">
+    <parent link="base_footprint" />
+    <child link="root" />
+    <origin xyz="0 0 0" rpy="0 0 0" />
+  </joint>
+  <link name="root"/>
   <joint name="base_link_joint" type="fixed">
-    <origin xyz="0.0 0 0" rpy="0 0 0" />
+    <origin xyz="0.0 0 0.4" rpy="0 0 0" />
     <parent link="base_footprint"/>
     <child link="agv_base_link" />
@@ -36,9 +40,8 @@
     <visual>
      <origin
-        xyz="-0.20 -0.445 0"
+        xyz="-0.213 -0.438 -0.4745"
         rpy="1.5708 0 1.5708"/>
       <geometry>
-      <mesh
-          filename="$(find kinova_description)/meshes/WMRM.STL" scale="0.001 0.001 0.001"/>
+        <mesh filename="$(find kinova_description)/meshes/WMRM.STL" scale="0.001 0.001 0.001"/>
       </geometry>
       <material
@@ -50,24 +53,31 @@
     <collision>
       <origin
-         xyz="0.32 0 0.25"
+         xyz="0 0 -0.4"
          rpy="0 0 0" />
       <geometry>
-        <box size="0.8 0.615 0.5" />
+        <mesh filename="$(find kinova_description)/meshes/collision.STL" scale="0.001 0.001 0.001"/>
+        <!-- <box size="0.8 0.615 0.5" /> -->
       </geometry>
     </collision>
   </link>
-  <link name="laser_link0"/>
-  <link name="laser_link1"/>
+  <joint name="laser_joint" type="fixed">
+    <origin xyz="0 0 -0.0745" rpy="0 0 0" />
+    <parent link="agv_base_link"/>
+    <child link="laser"/>
+  </joint>
+  <link name="laser"/>
   <joint name="laser0_joint" type="fixed">
-    <origin xyz="0.765 0.365 0.36" rpy="3.1419 0 3.9269" />
-    <parent link="agv_base_link"/>
-    <child link="laser_link0"/>
+    <origin xyz="0.818 0.415 0" rpy="0 0 0" />
+    <parent link="laser"/>
+    <child link="laser0"/>
   </joint>
-    <joint name="laser1_joint" type="fixed">
-    <origin xyz="-0.075 -0.365 0.36" rpy="3.14159 0 -0.7854" />
-    <parent link="agv_base_link"/>
-    <child link="laser_link1"/>
+  <joint name="laser1_joint" type="fixed">
+    <origin xyz="-0.07 -0.325 0" rpy="0 0 0" />
+    <parent link="laser"/>
+    <child link="laser1"/>
   </joint>
-  <gazebo reference="laser_link0">
+  <link name="laser0"/>
+  <link name="laser1"/>
+  <gazebo reference="laser0">
     <material>Gazebo/Blue</material>
     <turnGravityOff>false</turnGravityOff>
@@ -75,27 +85,27 @@
       <pose>0 0 0 0 0 0</pose>
       <visualize>false</visualize>
-      <update_rate>10</update_rate>
+      <update_rate>20</update_rate>
       <ray>
         <scan>
           <horizontal>
-            <samples>360</samples>
+            <samples>720</samples>
             <resolution>1</resolution>
-            <min_angle>${-M_PI}</min_angle>
+            <min_angle>${-M_PI/2}</min_angle>
             <max_angle>${M_PI}</max_angle>
           </horizontal>
         </scan>
         <range>
-          <min>0.10</min>
-          <max>10.0</max>
+          <min>0.05</min>
+          <max>12.0</max>
           <resolution>0.001</resolution>
         </range>
       </ray>
       <plugin name="gazebo_ros_head_hokuyo1_controller" filename="libgazebo_ros_laser.so">
-        <topicName>scan0</topicName>
-        <frameName>laser_link0</frameName>
+        <topicName>sim_scan0</topicName>
+        <frameName>sim_laser0</frameName>
       </plugin>
     </sensor>
   </gazebo>
-  <gazebo reference="laser_link1">
+  <gazebo reference="laser1">
     <material>Gazebo/Blue</material>
     <turnGravityOff>false</turnGravityOff>
@@ -103,23 +113,23 @@
       <pose>0 0 0 0 0 0</pose>
       <visualize>false</visualize>
-      <update_rate>10</update_rate>
+      <update_rate>20</update_rate>
       <ray>
         <scan>
           <horizontal>
-            <samples>360</samples>
+            <samples>720</samples>
             <resolution>1</resolution>
-            <min_angle>${-M_PI}</min_angle>
-            <max_angle>${M_PI}</max_angle>
+            <min_angle>${M_PI/2}</min_angle>
+            <max_angle>${2*M_PI}</max_angle>
           </horizontal>
         </scan>
         <range>
-          <min>0.10</min>
-          <max>10.0</max>
+          <min>0.05</min>
+          <max>12.0</max>
           <resolution>0.001</resolution>
         </range>
       </ray>
       <plugin name="gazebo_ros_head_hokuyo1_controller" filename="libgazebo_ros_laser.so">
-        <topicName>scan1</topicName>
-        <frameName>laser_link1</frameName>
+        <topicName>sim_scan1</topicName>
+        <frameName>sim_laser1</frameName>
       </plugin>
     </sensor>
@@ -136,14 +146,14 @@
   </plugin>
   </gazebo>
-    <xacro:include filename="$(find kinova_description)/urdf/j2s7s300.xacro"/>
-  <link name="root"/>
+  <xacro:include filename="$(find kinova_description)/urdf/j2s7s300.xacro"/>
+  <link name="robot_root"/>
   <!-- for gazebo
   <link name="world"/>-->
-  <joint name="connect_root_and_wheelchair" type="fixed">
-    <child link="root" />
+  <joint name="connect_robot_and_wheelchair" type="fixed">
+    <child link="robot_root" />
     <parent link="base_footprint" />
-    <origin xyz="0.715 0.32 0.513" rpy="0 0 1.5708" />
+    <origin xyz="0.6845 0.33 0.45" rpy="0 0 1.5708" />
   </joint>  -->
-  <xacro:property name="robot_root" value="root" />
+  <xacro:property name="robot_root" value="robot_root" />
   <xacro:j2s7s300  base_parent="${robot_root}"/>
 </robot>

Commit message: feat: 将gazebo仿真模型中kinova的位置上移5cm

File: src/kinova_description/urdf/j2s7s300_with_chair.xacro (robot description, xacro)
@@ -153,5 +153,5 @@
     <child link="robot_root" />
     <parent link="base_footprint" />
-    <origin xyz="0.6845 0.33 0.45" rpy="0 0 1.5708" />
+    <origin xyz="0.6845 0.33 0.5" rpy="0 0 1.5708" />
   </joint>  -->
   <xacro:property name="robot_root" value="robot_root" />
