Commit message: feat: 修改可达图的展示模型

File: src/kinova_description/urdf/wmrm.xacro (robot description, xacro)
@@ -43,5 +43,5 @@
         rpy="1.5708 0 1.5708"/>
       <geometry>
-        <mesh filename="$(find agv_description)/meshes/WMRM.STL" scale="0.001 0.001 0.001"/>
+        <mesh filename="package://kinova_description/meshes/WMRM.STL" scale="0.001 0.001 0.001"/>
       </geometry>
       <material
@@ -56,5 +56,5 @@
          rpy="0 0 0" />
       <geometry>
-        <mesh filename="$(find agv_description)/meshes/collision.STL" scale="0.001 0.001 0.001"/>
+        <mesh filename="package://kinova_description/meshes/collision.STL" scale="0.001 0.001 0.001"/>
         <!-- <box size="0.8 0.615 0.5" /> -->
       </geometry>

Commit message: feat: 修改了xacro文件中轮椅和机械臂基座的相对高度

File: src/kinova_description/urdf/wmrm.xacro (robot description, xacro)
@@ -153,5 +153,5 @@
     <child link="robot_root" />
     <parent link="base_footprint" />
-    <origin xyz="0.6845 0.33 0.5" rpy="0 0 1.5708" />
+    <origin xyz="0.6845 0.33 0.46" rpy="0 0 1.5708" />
   </joint>  -->
   <xacro:property name="robot_root" value="robot_root" />
